Commit message: Add files via upload

File: body.urdf (robot description, URDF)
Before this commit: robot robot, 9 links, 8 joints
Joints:
- joint BackLeg_BackLowerLeg: origin xyz=0.0 -1.0 0.0 rpy=0 0 0 -> xyz=0.0 -1.0 0.5 rpy=0 0 0
- joint FrontLeg_FrontLowerLeg: origin xyz=0.0 1.0 0.0 rpy=0 0 0 -> xyz=0.0 1.0 0.5 rpy=0 0 0
- joint LeftLeg_LeftLowerLeg: origin xyz=-1.0 0.0 0.0 rpy=0 0 0 -> xyz=-1.0 0.0 0.5 rpy=0 0 0
- joint RightLeg_RightLowerLeg: origin xyz=1.0 0.0 0.0 rpy=0 0 0 -> xyz=1.0 0.0 0.5 rpy=0 0 0
- joint Torso_BackLeg: origin xyz=0.0 -0.5 1.0 rpy=0 0 0 -> xyz=0.0 -0.5 2 rpy=0 0 0
- joint Torso_FrontLeg: origin xyz=0.0 0.5 1.0 rpy=0 0 0 -> xyz=0.0 0.5 2 rpy=0 0 0
- joint Torso_LeftLeg: origin xyz=-0.5 0.0 1.0 rpy=0 0 0 -> xyz=-0.5 0.0 2 rpy=0 0 0
- joint Torso_RightLeg: origin xyz=0.5 0.0 1.0 rpy=0 0 0 -> xyz=0.5 0.0 2 rpy=0 0 0
